File: High current 4x1 LED mux.sch (KiCad schematic (older format))
At the start: 120 parts, among them J1 Barrel_Jack_Switch, J10 Conn_01x24_Female, J2 Conn_01x02_Female, J3 8P8C_Shielded_x4, J4 Conn_01x03_Male, J5 Conn_01x03_Female, J6 Conn_01x08_Female, J7 Conn_01x03_Female, J8 Conn_01x05_Female, J9 Conn_01x24_Female, M1 Fan_4pin, Q1 SUM70060E, SW1 Pushbutton_with_LED, SW2 Pushbutton_with_LED, SW3 Pushbutton_with_LED, SW4 Pushbutton_with_LED, SW5 SW_SPDT, U1 12V boost, U12 Teensy3.6, U13 EL7457CSZ-T7, U2 SN74LV4T125PWR, U3 DPBW06F-05, U4 TMUX1204DGSR, U5 BDJ0GA5WEFJ-E2, U6 ADP7182AUJZ-1.8-R7, U7 LT6200CS8-10, U8 IRF9358TRPBF, U9 IRF9358TRPBF

Commit message: Preliminary layout
Parts:
- removed BZ1: CPT-2016-75-SMT-TR, Custom Footprints:SMT-0940-T-3V-R_9x9_alarm, symbol Custom_parts:CPT-2016-75-SMT-TR
- removed C1, C2, C3: 7500uF, Custom Footprints:CP_Elec_18x22-EEE-FK1C752SV, symbol Device:CP1_Small
- removed C10, C13, C14, C4, C5, C6, C7, C8: 47uF, Capacitor_SMD:C_1206_3216Metric, symbol Device:C_Small
- removed C11, C12, C21: 2200pF, Capacitor_SMD:C_0603_1608Metric, symbol Device:C_Small
- removed C15, C16, C17, C18, C19, C20, C22, C9: 2.2uF, Custom Footprints:0508_Capacitor, symbol Device:C_Small
- removed D1, D2, D3: BAT54BRW, Package_TO_SOT_SMD:SOT-363_SC-70-6, symbol Custom_parts:BAT54BRW
- removed D4: D_Zener, Diode_SMD:D_SOD-323, symbol Device:D_Zener
- removed D5: TVS_Diode, Custom Footprints:DO-214AA, symbol Device:D_Zener_Small_ALT
- removed H1, H10, H2, H4, H5, H6, H8: MountingHole_Pad, Custom Footprints:Ref_only, symbol Mechanical:MountingHole_Pad
- removed H3: MountingHole_Pad, Custom Footprints:NF-A9_with_standoffs_and_bolts, symbol Mechanical:MountingHole_Pad
- removed H7, H9: MountingHole_Pad, Custom Footprints:M2_standoff_ground_via, symbol Mechanical:MountingHole_Pad
- removed HS3, HS4: HS-PCB, Custom Footprints:Heatsink_910-40-2-23-2-B-0, symbol Mechanical:Heatsink
- removed J1: Barrel_Jack_Switch, Custom Footprints:DC-jack_54-00165, symbol Connector:Barrel_Jack_Switch
- removed J10, J9: Conn_01x24_Female, Custom Footprints:Ref_only, symbol Custom_parts:Conn_01x24_Female
- removed J2: Conn_01x02_Female, Custom Footprints:Wire_Pad, symbol Connector:Conn_01x02_Female
- removed J4: Conn_01x03_Male, Custom Footprints:Ref_only, symbol Custom_parts:Conn_01x03_Male
- removed J5, J7: Conn_01x03_Female, Custom Footprints:Ref_only, symbol Custom_parts:Conn_01x03_Female
- removed J6: Conn_01x08_Female, Custom Footprints:Ref_only, symbol Custom_parts:Conn_01x08_Female
- removed J8: Conn_01x05_Female, Custom Footprints:Ref_only, symbol Custom_parts:Conn_01x05_Female
- removed JP1: LED wire, Custom Footprints:L-Wire_Pad, symbol Device:Jumper_NO_Small
- removed JP2: Jumper_NC_Small, Resistor_SMD:R_2010_5025Metric, symbol Device:Jumper_NO_Small
- removed JP3, JP6: Jumper_NC_Small, Resistor_SMD:R_1206_3216Metric, symbol Device:Jumper_NC_Small
- removed JP4, JP5: Jumper_NC_Small, Custom Footprints:20A_shunt_5104, symbol Device:Jumper_NC_Small
- removed L1: 10uH, Inductor_SMD:L_1210_3225Metric, symbol pspice:INDUCTOR
- removed M1: Fan_4pin, Custom Footprints:4-pin_fan_SMD, symbol Motor:Fan_4pin
- removed Q1: SUM70060E, Package_TO_SOT_SMD:TO-263-2, symbol Device:Q_NMOS_GDS
- removed Q?: DMN32D2LDF-7, symbol Custom_parts:DMN32D2LDF-7
- removed R1, R2, R7: 12, Resistor_SMD:R_1210_3225Metric, symbol Device:R_Small
- removed R3, R4, R5, R6: 5, Custom Footprints:TO-252_resistor, symbol Device:R_Small
- removed RN1: 150, Custom Footprints:EXB-2HV151JV-1605x8, symbol Device:R_Pack08_Split
- removed RN2, RN4: 200, Resistor_SMD:R_Array_Convex_4x0612, symbol Device:R_Pack04_Split
- removed RN3: 4.7k, Custom Footprints:1506-EXB-2HV472JV-for_2_oz_pour, symbol Device:R_Pack08_Split
- removed RV1: R_POT, Custom Footprints:Pot_with_header, symbol Device:R_POT
- removed RV2, RV3: R_POT_TRIM, Custom Footprints:3224W-1-502E, symbol Device:R_POT_TRIM
- removed SW1, SW2, SW3, SW4: Pushbutton_with_LED, Custom Footprints:Pushbutton_LED-ELUMOATHQ3C12, symbol Custom_parts:Pushbutton_with_LED_-_ELUMOATHQ3C12
- removed SW5: SW_SPDT, Custom Footprints:1x5_header_SSM-105-L-SV-BE-LC, symbol Custom_parts:SW_SPDT-panel_ground
- removed TH1, TH2: Thermistor, Resistor_SMD:R_0603_1608Metric, symbol Device:Thermistor
- removed U1: 12V boost, Custom Footprints:12V_DC-DC_with_header_2117, symbol Regulator_Switching:R-78B1.2-2.0
- removed U12: Teensy3.6, Custom Footprints:Teensy_3_6_with_headers, symbol Custom_parts:Teensy3.6
- removed U13: EL7457CSZ-T7, Custom Footprints:EL7457CS, symbol Custom_parts:EL7457CSZ-T7
- removed U2: SN74LV4T125PWR, Custom Footprints:SN74LV4T125, symbol Custom_parts:SN74LV4T125PWR
- removed U3: DPBW06F-05, Custom Footprints:DPBW06F-05_with_header, symbol Custom_parts:DPBW06F-05
- removed U4: TMUX1204DGSR, Custom Footprints:TMUX1204DGSR, symbol Custom_parts:TMUX1204DGSR
- removed U5: BDJ0GA5WEFJ-E2, Custom Footprints:BDJ0GA5WEFJ-E2, symbol Custom_parts:BDJ0GA5WEFJ-E2
- removed U6: ADP7182AUJZ-1.8-R7, Package_TO_SOT_SMD:TSOT-23-5, symbol Custom_parts:ADP7182AUJZ-1.8-R7
- removed U7: LT6200CS8-10, Package_SO:SOIC-8_3.9x4.9mm_P1.27mm, symbol Custom_parts:LT6200CS8-10
- removed U8, U9: IRF9358TRPBF, Package_SO:SO-8_3.9x4.9mm_P1.27mm, symbol Custom_parts:SI9933CDY-T1-GE3
- added H1, H2, H3, H4: MountingHole, Custom Footprints:14-20_standoff, symbol Mechanical:MountingHole
- added Q2: DMN32D2LDF-7, Package_TO_SOT_SMD:SOT-353_SC-70-5, symbol Custom_parts:DMN32D2LDF-7
- gave numbers to parts that had none: 23
Connections:
- net labels removed: -0.25V_analog, -1.8V-analog, -5V, 10V-analog, 3.3V, 5V, 5V_fan_PWM, A-D_input_1, A-D_input_2, A-D_input_3, A-D_input_4, Analog_select, Button1, Button2, Button3, Button4, External_5V_PWM1, External_5V_PWM2, External_5V_PWM3, External_thermistor, Interline_PWM, Internal_fan_PWM, Isense, Isense_internal, LED1, LED2, LED3, LED4, LED_pot, MOSFET_temp, NC1, NC2, NC3, NC4, NC5, NC6, NC7, NC8, OA_input, Over_temp_alarm1, Over_temp_alarm2, Relay1, Relay2, Relay3, Relay4, Resistor_temp, SCL0, SDA0, Toggle_switch, Vcc, Vin, external_analog, internal_analog
- wire segments 260 -> 58
- no-connect marks 58 -> 8
Other:
- note removed: "**"
- note removed: "-------ADC0------"
- note removed: "--ADC1--"
- note removed: "3.3V clamp for external analog\nMax voltage: +6V/-3V"
- note removed: "4-channel analog/digital IO with 0-3.3V clamp"
- note removed: "4-pin 92mm fan"
- note removed: "4x momentary pushbuttons with indicator LEDs"
- note removed: "ADC0"
- note removed: "ADC1"
- note removed: "Boost - Vin (3V - 12V) to 12V DC"
- note removed: "Constant Current LED Driver with Compensation\n\n"
- note removed: "ISOLATED: 12V to split +/- 5V"
- note removed: "Inputs and Outputs\n"
- note removed: "Isense resistor and MOSFET\nthermitor temperature monitoring"
- note removed: "LED High-Side Gate Driver 4x1 Mux\n\n"
- note removed: "LED bypass capacitor array"
- note removed: "Manual/Auto toggle switch"
- note removed: "Op-amp input 4x1 mux"
- note removed: "Op-amp linear reagulator split supply: \n12V/-5V to clean 10V/-1.8V"
- note removed: "Optional bypass jumper"
- note removed: "Overheat alarm"
- note removed: "Pot to adjust LED intensity"
- note removed: "Teensy 3.6 180 MHz Microcontroller"
- note removed: "Thermal Management\n"
- note removed: "Voltage Rails: 12V, 10V, 5V, -0.25V, -1.8V, -5V\n\n"
- note removed: "https://forum.pjrc.com/attachment.php?attachmentid=10666&d=1495536536"
- note removed: "small negative \nreference voltage \nso that LED turns \noff with op-amp \ninput bias"
- moved on the sheet: C1, D1, D2, D3, D4, HS1, HS2, J1, J2, J3A, J3B, J3C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
