File: High current 4x1 LED mux.sch (KiCad schematic (older format))
At the start: 34 parts, among them J1 Barrel_Jack_Switch, J2 Conn_01x04_Female, J3 8P8C_Shielded_x4, M1 Fan_4pin, M2 Fan_4pin, M3 Fan_4pin, M4 Fan_4pin, Q1 DMN32D2LDF-7, Q2 DMN32D2LDF-7, Q3 SUM70060E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

Commit message: Add Gerber files
Parts:
- renumbered Q3 to Q1, Q4 to Q2, Q5 to Q3, Q6 to Q4, Q1 to Q5, Q2 to Q6
Changed lines of the file:
@@
 $EndComp
 $Comp
-L Device:Q_NMOS_GDS Q3
+L Device:Q_NMOS_GDS Q1
 U 1 1 617829C7
 P 4700 3850
-F 0 "Q3" H 4904 3896 50  0000 L CNN
+F 0 "Q1" H 4904 3896 50  0000 L CNN
 F 1 "SUM70060E" H 4904 3805 50  0000 L CNN
 F 2 "Package_TO_SOT_SMD:TO-263-2" H 4900 3950 50  0001 C CNN
@@
 LED-
 $Comp
-L Device:Q_NMOS_GDS Q4
+L Device:Q_NMOS_GDS Q2
 U 1 1 617AD81E
 P 4700 4350
-F 0 "Q4" H 4904 4396 50  0000 L CNN
+F 0 "Q2" H 4904 4396 50  0000 L CNN
 F 1 "SUM70060E" H 4904 4305 50  0000 L CNN
 F 2 "Package_TO_SOT_SMD:TO-263-2" H 4900 4450 50  0001 C CNN
@@
 LED-
 $Comp
-L Device:Q_NMOS_GDS Q5
+L Device:Q_NMOS_GDS Q3
 U 1 1 617BC877
 P 4700 4850
-F 0 "Q5" H 4904 4896 50  0000 L CNN
+F 0 "Q3" H 4904 4896 50  0000 L CNN
 F 1 "SUM70060E" H 4904 4805 50  0000 L CNN
 F 2 "Package_TO_SOT_SMD:TO-263-2" H 4900 4950 50  0001 C CNN
@@
 LED-
 $Comp
-L Device:Q_NMOS_GDS Q6
+L Device:Q_NMOS_GDS Q4
 U 1 1 617CC07E
 P 4700 5350
-F 0 "Q6" H 4904 5396 50  0000 L CNN
+F 0 "Q4" H 4904 5396 50  0000 L CNN
 F 1 "SUM70060E" H 4904 5305 50  0000 L CNN
 F 2 "Package_TO_SOT_SMD:TO-263-2" H 4900 5450 50  0001 C CNN
@@
 $EndComp
 $Comp
-L Custom_parts:DMN32D2LDF-7 Q1
+L Custom_parts:DMN32D2LDF-7 Q5
 U 1 1 6186157F
 P 4100 6600
-F 0 "Q1" H 4200 7197 60  0000 C CNN
+F 0 "Q5" H 4200 7197 60  0000 C CNN
 F 1 "DMN32D2LDF-7" H 4200 7091 60  0000 C CNN
 F 2 "Package_TO_SOT_SMD:SOT-353_SC-70-5" H 3750 5800 60  0001 L CNN
@@
 $EndComp
 $Comp
-L Custom_parts:DMN32D2LDF-7 Q2
+L Custom_parts:DMN32D2LDF-7 Q6
 U 1 1 617D9FE3
 P 4100 7550
-F 0 "Q2" H 4200 8147 60  0000 C CNN
+F 0 "Q6" H 4200 8147 60  0000 C CNN
 F 1 "DMN32D2LDF-7" H 4200 8041 60  0000 C CNN
 F 2 "Package_TO_SOT_SMD:SOT-353_SC-70-5" H 3750 6750 60  0001 L CNN

Commit message: Bigger spacing on 100V planes to prevent shorting
Parts:
- Q5, Q6: symbol Custom_parts:DMN32D2LDF-7 -> High-current-4x1-LED-mux-rescue:DMN32D2LDF-7-Custom_parts
- U1: symbol High-current-4x1-LED-mux-rescue:MIC4468ZWM-TR-Custom_parts-High-current-1x4-LED-mux-rescue -> High-current-4x1-LED-mux-rescue:MIC4468ZWM-TR-Custom_parts-High-current-1x4-LED-mux-rescue-High-current-4x1-LED-mux-res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
Changed lines of the file:
@@
 LED-
 $Comp
-L High-current-4x1-LED-mux-rescue:MIC4468ZWM-TR-Custom_parts-High-current-1x4-LED-mux-rescue U1
+L High-current-4x1-LED-mux-rescue:MIC4468ZWM-TR-Custom_parts-High-current-1x4-LED-mux-rescue-High-current-4x1-LED-mux-rescue U1
 U 1 1 617F4C37
 P 3250 4250
@@
 $EndComp
 $Comp
-L Custom_parts:DMN32D2LDF-7 Q5
+L High-current-4x1-LED-mux-rescue:DMN32D2LDF-7-Custom_parts Q5
 U 1 1 6186157F
 P 4100 6600
@@
 $EndComp
 $Comp
-L Custom_parts:DMN32D2LDF-7 Q6
+L High-current-4x1-LED-mux-rescue:DMN32D2LDF-7-Custom_parts Q6
 U 1 1 617D9FE3
 P 4100 7550
